Commit message: dd

File: Task_Workspace/simulation_packages/env_sim/urdf/simplified_ur5_1.urdf (robot description, URDF)
Before this commit: robot ur5, 14 links, 13 joints
Links:
- link ur5_base_link: geometry collision cylinder length=0.12 radius=0.075; visual cylinder length=0.12 radius=0.075
- link ur5_forearm_link: geometry collision box size=0.39225 0.1 0.1; visual box size=0.39225 0.1 0.1
- link ur5_shoulder_link: geometry collision cylinder length=0.12 radius=0.075; visual cylinder length=0.12 radius=0.075
- link ur5_upper_arm_link: geometry collision box size=0.425 0.1 0.1; visual box size=0.425 0.1 0.1
- link ur5_wrist_1_link: geometry collision cylinder length=0.1 radius=0.06; visual cylinder length=0.1 radius=0.06
- link ur5_wrist_2_link: geometry collision cylinder length=0.1 radius=0.06; visual cylinder length=0.1 radius=0.06
- link ur5_wrist_3_link: geometry collision cylinder length=0.08 radius=0.045; visual cylinder length=0.08 radius=0.045
